File: alt-Lab2/arduino_Uno_ref/arduino_uno_mod.brd (EAGLE design)
At the start: 68.6 x 53.3 mm, 63 parts, among them IC1 MC33269ST-5.0T3, IC2 MC33269D-5.0, Q1 16MHz, Q2 16MHz, Q3 BSS101, T1 FDN304V, U1 LM358D, U2 LP2985-33DBVR, U3 ATMEGA8U2-MU, X1 DC21MMX, Y1 16MHz, Y2 16MHz

Commit message: pre-merge commit
Parts:
- moved L2 84.1 mm to (51.4, 41.9)
- moved C13 81.4 mm to (51.4, 36.8), turned to 180 degrees
- moved D2 81.4 mm to (40.0, 38.7), turned to 270 degrees
- moved R4 16.5 mm to (-22.9, -27.9)
Changed lines of the file:
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@@
 <attribute name="VALUE" x="-7.62" y="-40.005" size="1.27" layer="27" ratio="10"/>
 </element>
-<element name="D2" library="diode" library_urn="urn:adsk.eagle:library:210" package="DO41-10" package3d_urn="urn:adsk.eagle:package:43336/1" value="1N4004" x="-7.62" y="-27.305" smashed="yes">
-<attribute name="NAME" x="-9.652" y="-25.654" size="1.27" layer="25" ratio="10"/>
-<attribute name="POPULARITY" value="82" x="-7.62" y="-24.765" size="1.778" layer="27" display="off"/>
-<attribute name="VALUE" x="-9.652" y="-30.099" size="1.27" layer="27" ratio="10"/>
+<element name="D2" library="diode" library_urn="urn:adsk.eagle:library:210" package="DO41-10" package3d_urn="urn:adsk.eagle:package:43336/1" value="1N4004" x="40.005" y="38.735" smashed="yes" rot="R270">
+<attribute name="NAME" x="41.656" y="40.767" size="1.27" layer="25" ratio="10" rot="R270"/>
+<attribute name="POPULARITY" value="82" x="42.545" y="38.735" size="1.778" layer="27" rot="R270" display="off"/>
+<attribute name="VALUE" x="37.211" y="40.767" size="1.27" layer="27" ratio="10" rot="R270"/>
 </element>
-<element name="R4" library="rcl" library_urn="urn:adsk.eagle:library:334" package="0207/10" package3d_urn="urn:adsk.eagle:package:23491/2" value="" x="-7.62" y="-34.29" smashed="yes">
-<attribute name="NAME" x="-10.668" y="-32.766" size="1.27" layer="25" ratio="10"/>
-<attribute name="POPULARITY" value="81" x="-7.62" y="-31.75" size="1.778" layer="27" display="off"/>
-<attribute name="SPICEPREFIX" value="R" x="-7.62" y="-31.75" size="1.778" layer="27" display="off"/>
-<attribute name="VALUE" x="-9.8806" y="-34.925" size="1.27" layer="27" ratio="10"/>
+<element name="R4" library="rcl" library_urn="urn:adsk.eagle:library:334" package="0207/10" package3d_urn="urn:adsk.eagle:package:23491/2" value="" x="-22.86" y="-27.94" smashed="yes">
+<attribute name="NAME" x="-25.908" y="-26.416" size="1.27" layer="25" ratio="10"/>
+<attribute name="POPULARITY" value="81" x="-22.86" y="-25.4" size="1.778" layer="27" display="off"/>
+<attribute name="SPICEPREFIX" value="R" x="-22.86" y="-25.4" size="1.778" layer="27" display="off"/>
+<attribute name="VALUE" x="-25.1206" y="-28.575" size="1.27" layer="27" ratio="10"/>
 </element>
-<element name="C13" library="capacitor-wima" library_urn="urn:adsk.eagle:library:116" package="C2.5-2" package3d_urn="urn:adsk.eagle:package:5415/1" value="" x="1.27" y="-27.305" smashed="yes">
-<attribute name="NAME" x="-0.381" y="-25.781" size="1.27" layer="25" ratio="10"/>
-<attribute name="POPULARITY" value="28" x="-10.795" y="-36.83" size="1.778" layer="27" display="off"/>
-<attribute name="VALUE" x="-0.381" y="-30.099" size="1.27" layer="27" ratio="10"/>
+<element name="C13" library="capacitor-wima" library_urn="urn:adsk.eagle:library:116" package="C2.5-2" package3d_urn="urn:adsk.eagle:package:5415/1" value="" x="51.435" y="36.83" smashed="yes" rot="R180">
+<attribute name="NAME" x="53.086" y="35.306" size="1.27" layer="25" ratio="10" rot="R180"/>
+<attribute name="POPULARITY" value="28" x="63.5" y="46.355" size="1.778" layer="27" rot="R180" display="off"/>
+<attribute name="VALUE" x="53.086" y="39.624" size="1.27" layer="27" ratio="10" rot="R180"/>
 </element>
-<element name="L2" library="inductors" library_urn="urn:adsk.eagle:library:243" package="LBC15" package3d_urn="urn:adsk.eagle:package:15085/1" value="LBC15" x="-4.445" y="-20.955" smashed="yes">
-<attribute name="NAME" x="-10.16" y="-17.907" size="1.27" layer="25" ratio="10"/>
-<attribute name="POPULARITY" value="0" x="-4.445" y="-43.18" size="1.778" layer="27" display="off"/>
-<attribute name="SPICEPREFIX" value="L" x="-4.445" y="-43.18" size="1.778" layer="27" display="off"/>
-<attribute name="VALUE" x="-9.525" y="-22.098" size="1.27" layer="27" ratio="10"/>
+<element name="L2" library="inductors" library_urn="urn:adsk.eagle:library:243" package="LBC15" package3d_urn="urn:adsk.eagle:package:15085/1" value="LBC15" x="51.435" y="41.91" smashed="yes">
+<attribute name="NAME" x="45.72" y="44.958" size="1.27" layer="25" ratio="10"/>
+<attribute name="POPULARITY" value="0" x="51.435" y="19.685" size="1.778" layer="27" display="off"/>
+<attribute name="SPICEPREFIX" value="L" x="51.435" y="19.685" size="1.778" layer="27" display="off"/>
+<attribute name="VALUE" x="46.355" y="40.767" size="1.27" layer="27" ratio="10"/>
 </element>
 <element name="J1" library="jumper" library_urn="urn:adsk.eagle:library:252" package="04C" package3d_urn="urn:adsk.eagle:package:15506/1" value="" x="-10.795" y="-43.815" smashed="yes">
@@
 <wire x1="11.15" y1="15.119" x2="11.43" y2="12.7" width="0" layer="19" extent="1-1"/>
 <wire x1="43.688" y1="50.673" x2="28.956" y2="44.45" width="0" layer="19" extent="1-1"/>
-<wire x1="2.54" y1="-27.305" x2="8.6868" y2="3.302" width="0" layer="19" extent="1-1"/>
-<wire x1="-2.54" y1="-27.305" x2="2.54" y2="-27.305" width="0" layer="19" extent="1-1"/>
-<wire x1="-12.7" y1="-34.29" x2="-2.54" y2="-27.305" width="0" layer="19" extent="1-1"/>
+<wire x1="50.165" y1="36.83" x2="8.6868" y2="3.302" width="0" layer="19" extent="1-1"/>
+<wire x1="40.005" y1="33.655" x2="50.165" y2="36.83" width="0" layer="19" extent="1-1"/>
+<wire x1="-27.94" y1="-27.94" x2="40.005" y2="33.655" width="0" layer="19" extent="1-1"/>
 </signal>
 <signal name="AREF">
@@
 <contactref element="ZIC1" pad="13"/>
 <contactref element="IOL" pad="8"/>
-<wire x1="46.101" y1="35.433" x2="46.101" y2="48.641" width="0.4064" layer="16"/>
-<wire x1="46.101" y1="48.641" x2="45.72" y2="49.022" width="0.4064" layer="16"/>
-<wire x1="45.72" y1="49.022" x2="45.72" y2="50.8" width="0.4064" layer="16"/>
+<wire x1="45.72" y1="35.052" x2="45.72" y2="50.8" width="0.4064" layer="16"/>
 <wire x1="32.385" y1="20.193" x2="32.385" y2="21.717" width="0.4064" layer="16"/>
-<wire x1="32.385" y1="21.717" x2="46.101" y2="35.433" width="0.4064" layer="16"/>
+<wire x1="32.385" y1="21.717" x2="45.72" y2="35.052" width="0.4064" layer="16"/>
 </signal>
 <signal name="IO8">
@@
 <contactref element="L2" pad="1"/>
 <contactref element="D2" pad="C"/>
-<wire x1="-12.7" y1="-27.305" x2="-9.525" y2="-38.735" width="0" layer="19" extent="1-1"/>
-<wire x1="-12.065" y1="-20.955" x2="-12.7" y2="-27.305" width="0" layer="19" extent="1-1"/>
+<wire x1="40.005" y1="43.815" x2="-9.525" y2="-38.735" width="0" layer="19" extent="1-1"/>
+<wire x1="43.815" y1="41.91" x2="40.005" y2="43.815" width="0" layer="19" extent="1-1"/>
 </signal>
 <signal name="BCO">
@@
 <contactref element="R4" pad="2"/>
 <contactref element="J2" pad="2"/>
-<wire x1="-2.54" y1="-34.29" x2="-8.89" y2="-48.26" width="0" layer="19" extent="1-1"/>
-<wire x1="0" y1="-27.305" x2="-2.54" y2="-34.29" width="0" layer="19" extent="1-1"/>
-<wire x1="3.175" y1="-20.955" x2="0" y2="-27.305" width="0" layer="19" extent="1-1"/>
+<wire x1="-17.78" y1="-27.94" x2="-8.89" y2="-48.26" width="0" layer="19" extent="1-1"/>
+<wire x1="52.705" y1="36.83" x2="-17.78" y2="-27.94" width="0" layer="19" extent="1-1"/>
+<wire x1="59.055" y1="41.91" x2="52.705" y2="36.83" width="0" layer="19" extent="1-1"/>
 </signal>
 <signal name="IAD0">
